File: reciever.kicad_sch (KiCad schematic)
At the start: 0 parts

Commit message: updatged schematics
Parts:
- added C21, C22, C23: 4.7muF, Capacitor_SMD:C_1206_3216Metric_Pad1.33x1.80mm_HandSolder, symbol Device:C
- added D2: LED, symbol Device:LED
- added IC2: SKY65405-21, SamacSys_Parts:SKY6540521, symbol SamacSys_Parts:SKY65405-21
- added IC6: RMS-30+, SamacSys_Parts:RMS30, symbol SamacSys_Parts:RMS-30+
- added J4, J5: Conn_Coaxial_x2, symbol Connector:Conn_Coaxial_x2
- added J6: USB_A, Connector_USB:USB3_A_Molex_48393-001, symbol Connector:USB_A
- added R12: 499, Resistor_SMD:R_0612_1632Metric_Pad1.18x3.40mm_HandSolder, symbol Device:R
- added R13: 33.2k, Resistor_SMD:R_0612_1632Metric_Pad1.18x3.40mm_HandSolder, symbol Device:R
- added R14: 200k, Resistor_SMD:R_0612_1632Metric_Pad1.18x3.40mm_HandSolder, symbol Device:R
- added R15: 453k, Resistor_SMD:R_0612_1632Metric_Pad1.18x3.40mm_HandSolder, symbol Device:R
- added R16: 49.9k, Resistor_SMD:R_0612_1632Metric_Pad1.18x3.40mm_HandSolder, symbol Device:R
- added R2: R, Resistor_SMD:R_0612_1632Metric_Pad1.18x3.40mm_HandSolder, symbol Device:R
- added U3: LT3042xMSE, Package_SO:MSOP-10-1EP_3x3mm_P0.5mm_EP1.68x1.88mm, symbol Regulator_Linear:LT3042xMSE
Connections:
- new net: R14.2, U3.4 (PG)
- new net: R12.2, U3.5 (ILIM)
- new net: R15.1, R16.2, U3.6 (PGFB)
- new net: C22.1, R13.2, U3.7 (SET)
- new net: IC6.5 (IF), J5.2 (IN2)
- new net: IC2.3 (RF_IN), J4.2 (IN2)
- new net: D2.1 (K), R2.1
- new net: IC2.4 (RF_OUT), IC6.4 (RF)
- new net +3.3V: C23.1, R15.2, U3.10 (OUT), U3.9 (OUTS)
- new net +5V: C21.1, D2.2 (A), IC2.1 (V_ENABLE_), IC2.6 (VCC), J6.1 (VBUS), R14.1, U3.1 (IN), U3.2 (IN), U3.3 (EN/UV)
- new net GND: C21.2, C22.2, C23.2, IC2.2 (GND_1), IC2.5 (GND_2), IC2.7 (GND_3), IC6.2 (GROUND_1), IC6.3 (GROUND_2), IC6.6 (GROUND_3), J4.3 (EXT), J5.3 (EXT), J6.4 (GND), J6.SH (Shield), R12.1, R13.1, R16.1, R2.2, U3.11 (GND), U3.8 (GND)
- new net Oscillator Output: IC6.1 (LO)
Other:
- title: (none) -> Reciever

Commit message: updated schematics
Parts:
- J4, J5: footprint (none) -> Connector_Coaxial:SMA_Amphenol_132289_EdgeMount
Changed lines of the file:
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@@
 			)
 		)
-		(property "Footprint" ""
+		(property "Footprint" "Connector_Coaxial:SMA_Amphenol_132289_EdgeMount"
 			(at 237.49 66.04 0)
 			(hide yes)
@@
 			)
 		)
-		(property "Footprint" ""
+		(property "Footprint" "Connector_Coaxial:SMA_Amphenol_132289_EdgeMount"
 			(at 52.07 86.36 0)
 			(hide yes)
